Commit message: add laser to sim and gazebo_control

File: urdf/src/my_robot/description/materials.xacro (robot description, xacro)
@@ -9,3 +9,6 @@
     <color rgba="0.2 0.2 1 1"/>
   </material>
+    <material name="black">
+    <color rgba="0 0 0 1"/>
+  </material>
 </xacro:macro>

File: urdf/src/my_robot/description/mrobot.urdf.xacro (robot description, xacro)
@@ -3,12 +3,10 @@
   <xacro:include filename="materials.xacro"/>
   <xacro:include filename="robot_core.xacro"/>
+  <xacro:include filename="gazebo_control.xacro"/>
+  <xacro:include filename="laser_core.xacro"/>
   <!-- instantiate -->
   <robot_core/>
   <materials/>
-<!-- ================= GAZEBO ================= -->
-  <gazebo>
-    <plugin
-      name="gazebo_ros_control"
-      filename="libgazebo_ros2_control.so"/>
-  </gazebo>
+  <diff_drive/>
+  <laser_core/>
 </robot>

File: urdf/src/my_robot/description/robot_core.xacro (robot description, xacro)
@@ -51,4 +51,7 @@
     </collision>
   </link>
+  <gazebo reference="chassis">
+      <material>Gazebo/White</material>
+  </gazebo>
   <!-- LEFT WHEEL -->
   <joint name="left_wheel_joint" type="continuous">
@@ -57,5 +60,11 @@
     <origin xyz="0 0.175 0" rpy="-${pi/2} 0 0"/>
     <axis xyz="0 0 1"/>
+    <dynamics damping="1.0" friction="0.1"/>
   </joint>
+  <gazebo reference="left_wheel">
+      <material>Gazebo/Blue</material>
+      <mu1 value="1.0"/>
+      <mu2 value="1.0"/>
+  </gazebo>
   <link name="left_wheel">
     <visual>
@@ -91,5 +100,11 @@
     <origin xyz="0 -0.175 0" rpy="${pi/2} 0 0"/>
     <axis xyz="0 0 -1"/>
+    <dynamics damping="1.0" friction="0.1"/>
   </joint>
+  <gazebo reference="right_wheel">
+      <material>Gazebo/Blue</material>
+      <mu1 value="1.0"/>
+      <mu2 value="1.0"/>
+  </gazebo>
   <link name="right_wheel">
     <visual>
@@ -125,8 +140,13 @@
       <origin xyz="0.24 0 0" rpy="0 0 0"/>
   </joint>
+  <gazebo reference="caster_wheel">
+      <material>Gazebo/Black</material>
+      <mu1 value="0.001"/>
+      <mu2 value="0.001"/>
+  </gazebo>
   <link name="caster_wheel">
       <visual>
           <geometry>
-              <sphere radius="0.05" />
+              <sphere radius="0.04" />
           </geometry>
           <material name="black"/>
@@ -136,5 +156,5 @@
         <origin xyz="0.0 0.0 0.0" rpy="0.0 0.0 0.0"/>
         <geometry>
-          <sphere radius="0.05"/>
+          <sphere radius="0.04"/>
         </geometry>
       </collision>
