Commit message: simulation robot and control with nav2

File: urdf/src/my_robot/description/laser_core.xacro (robot description, xacro)
@@ -6,5 +6,5 @@
     <inertial_cylinder/>
     <joint name="laser_joint" type="fixed">
-        <parent link="chassis"/>
+        <parent link="base_link"/>
         <child link="laser_frame"/>
         <origin xyz="0.1 0 0.175" rpy="0 0 0"/>

File: urdf/src/my_robot/description/robot_core.xacro (robot description, xacro)
@@ -29,4 +29,12 @@
   <!-- BASE -->
   <link name="base_link"/>
+  <!-- Base_footprint -->
+  <joint name="base_footprint_joint" type="fixed">
+    <parent link="base_link"/>
+    <child link="base_footprint"/>
+    <origin xyz="0.0 0.0 0.0" rpy="0.0 0.0 0.0"/>
+  </joint>
+  <link name="base_footprint">
+  </link>
   <!-- CHASSIS -->
   <joint name="chassis_joint" type="fixed">
