Commit message: build excutor file to solve ik

File: Project/scara_ws/src/scara_robot/description/core.xacro (robot description, xacro)
@@ -93,5 +93,5 @@
     <!-- Joint 4 -->
     <joint name="joint_4" type="fixed">
-        <origin xyz="0.1 0.0 0.0" rpy="0.0 0.0 0.0"/>
+        <origin xyz="0.0 0.0 0.0" rpy="0.0 0.0 0.0"/>
         <parent link="link_3"/>
         <child link="link_4"/>
@@ -155,8 +155,8 @@
     <!-- Joint 6 -->
     <joint name="joint_6" type="prismatic">
-        <origin xyz="0.0 0.0 0.0" rpy="0.0 0.0 0.0"/>
+        <origin xyz="0 0 0" rpy="${pi} 0 0"/>
         <parent link="link_5"/>
         <child link="link_6"/>
-        <axis xyz="0.0 0.0 -1.0"/>
+        <axis xyz="0.0 0.0 1.0"/>
         <limit lower="0" upper="0.5" effort="10.0" velocity="1.0"/>
     </joint>

File: Project/scara_ws/src/scara_robot/description/ros2_control.xacro (robot description, xacro)
@@ -1,24 +1,22 @@
-<xacro:macro name="control" xmlns:xacro="http://www.ros.org/wiki/xacro">
-    <ros2_control type="system">
+<xacro:macro name="control" xmlns:xacro="http://www.ros.org/wiki/xacro" >
+  <ros2_control name="ScaraSystem" type="system">
     <hardware>
-        <!-- Fake hardware để test RViz -->
-        <plugin>mock_components/GenericSystem</plugin>
+      <plugin>mock_components/GenericSystem</plugin>
     </hardware>
     <joint name="joint_1">
-        <command_interface name="position"/>
-        <state_interface name="position"/>
-    </joint>
-    <joint name="joint_2">
-        <command_interface name="position"/>
-        <state_interface name="position"/>
+      <command_interface name="position"/>
+      <state_interface name="position"/>
+      <state_interface name="velocity"/>
     </joint>
     <joint name="joint_3">
-        <command_interface name="position"/>
-        <state_interface name="position"/>
+      <command_interface name="position"/>
+      <state_interface name="position"/>
+      <state_interface name="velocity"/>
     </joint>
     <joint name="joint_6">
-        <command_interface name="position"/>
-        <state_interface name="position"/>
+      <command_interface name="position"/>
+      <state_interface name="position"/>
+      <state_interface name="velocity"/>
     </joint>
-    </ros2_control>
+  </ros2_control>
 </xacro:macro>

File: Project/scara_ws/src/scara_robot/description/scara.urdf.xacro (robot description, xacro)
@@ -1,8 +1,7 @@
 <?xml version="1.0"?>
 <robot xmlns:xacro="http://www.ros.org/wiki/xacro" name="scara_3dof">
-       <xacro:include filename="core.xacro"/>
-        <xacro:include filename="ros2_control.xacro"/>
-       <!-- instantiate -->
-       <scara_core/>
-       <control/>
+  <xacro:include filename="core.xacro"/>
+  <xacro:include filename="ros2_control.xacro"/>
+  <scara_core/>
+  <control/>
 </robot>
